File: audio.kicad_sch (KiCad schematic)
At the start: 29 parts, among them J5 1775443-2, U14 TAS5805MPWPR

Commit message: v2-fix: issue #53 fixes on the v2 hardware (XMOS 0.9V buck, Voice PE I2S roles, U12, JTAG header, TAS5805M ADR, LED level shift, routing bugs)
Based on 7de6eec (v2 hardware), without the ESP32-C6. See CHANGES-v2fix.md for the full list, references and known limitations. Untested candidate: needs layout review before fabrication.
Parts:
- R70: value 0R -> 15k; LCSC Part # (none) -> C25756; Manufacturer Part (none) -> 0402WGF1502TCE
- U14: LCSC Part # (none) -> C478472; Manufacturer Part (none) -> TAS5805MPWPR
Connections:
- net DGND: no longer R70.1
- net DVDD: now also R70.1
Changed lines of the file:
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@@
 	(wire
 		(pts
-			(xy 67.31 88.9) (xy 63.5 88.9)
-		)
-		(stroke
-			(width 0)
-			(type default)
-		)
-	)
-	(wire
-		(pts
 			(xy 147.32 129.54) (xy 149.86 129.54)
 		)
@@
 	(wire
 		(pts
-			(xy 63.5 88.9) (xy 63.5 91.44)
-		)
-		(stroke
-			(width 0)
-			(type default)
-		)
-	)
-	(wire
-		(pts
 			(xy 54.61 160.02) (xy 54.61 154.94)
 		)
@@
 			)
 		)
-		(property "Value" "0R"
+		(property "Value" "15k"
 			(at 75.184 87.376 90)
 			(effects
@@
 			)
 		)
-		(property "Description" "Resistor"
+		(property "Description" "TAS5805M ADR: 15k to DVDD = I2C 0x2D"
 			(at 71.12 88.9 0)
 			(effects
@@
 			)
 		)
+		(property "Manufacturer Part" "0402WGF1502TCE" (at 71.12 88.9 0) (effects (font (size 1.27 1.27)) (hide yes)))
+		(property "LCSC Part #" "C25756" (at 71.12 88.9 0) (effects (font (size 1.27 1.27)) (hide yes)))
 		(pin "1"
 		)
@@
 	)
 	(symbol
-		(lib_id "power:GND")
-		(at 63.5 91.44 0)
-		(unit 1)
-		(exclude_from_sim no)
-		(in_bom yes)
-		(on_board yes)
-		(dnp no)
-		(fields_autoplaced yes)
-		(property "Reference" "#PWR0153"
-			(at 63.5 97.79 0)
-			(effects
-				(font
-					(size 1.27 1.27)
-				)
-				(hide yes)
-			)
-		)
-		(property "Value" "GNDA"
-			(at 63.5 96.52 0)
-			(effects
-				(font
-					(size 1.27 1.27)
-				)
-			)
-		)
-		(property "Footprint" ""
-			(at 63.5 91.44 0)
-			(effects
-				(font
-					(size 1.27 1.27)
-				)
-				(hide yes)
-			)
-		)
-		(property "Datasheet" ""
-			(at 63.5 91.44 0)
-			(effects
-				(font
-					(size 1.27 1.27)
-				)
-				(hide yes)
-			)
-		)
-		(property "Description" "Power symbol creates a global label with name \"GND\" , ground"
-			(at 63.5 91.44 0)
-			(effects
-				(font
-					(size 1.27 1.27)
-				)
-				(hide yes)
-			)
-		)
-		(pin "1"
-		)
-		(instances
-			(project ""
-				(path "/204e071a-14ed-47a0-be54-332ac2b951cf/62ce711e-2967-4164-94ee-cdd918e5185e"
-					(reference "#PWR0153")
-					(unit 1)
-				)
-			)
-		)
-	)
-	(symbol
 		(lib_id "Device:C")
 		(at 193.04 59.69 0)
@@
 			)
 		)
+		(property "LCSC Part #" "C478472" (at 129.54 99.06 0) (effects (font (size 1.27 1.27)) (hide yes)))
+		(property "Manufacturer Part" "TAS5805MPWPR" (at 129.54 99.06 0) (effects (font (size 1.27 1.27)) (hide yes)))
 		(pin "23"
 		)
@@
 		)
 	)
+	(wire (pts (xy 67.31 88.9) (xy 63.5 88.9)) (stroke (width 0) (type default)))
+	(symbol
+		(lib_id "New_Library:PVDD1")
+		(at 63.5 88.9 90)
+		(unit 1)
+		(exclude_from_sim no)
+		(in_bom yes)
+		(on_board yes)
+		(dnp no)
+		(property "Reference" "#PWR0950" (at 63.5 83.9 0) (effects (font (size 1.27 1.27)) (hide yes)))
+		(property "Value" "DVDD" (at 63.5 93.9 0) (effects (font (size 1.27 1.27))))
+		(property "Footprint" "" (at 63.5 88.9 0) (effects (font (size 1.27 1.27)) (hide yes)))
+		(property "Datasheet" "~" (at 63.5 88.9 0) (effects (font (size 1.27 1.27)) (hide yes)))
+		(pin "1")
+		(instances (project "nest-mini-v2-drop-in-pcb" (path "/204e071a-14ed-47a0-be54-332ac2b951cf/62ce711e-2967-4164-94ee-cdd918e5185e" (reference "#PWR0950") (unit 1))))
+	)
 )
