File: leds.kicad_sch (KiCad schematic)
At the start: 12 parts

Commit message: v2-fix: issue #53 fixes on the v2 hardware (XMOS 0.9V buck, Voice PE I2S roles, U12, JTAG header, TAS5805M ADR, LED level shift, routing bugs)
Based on 7de6eec (v2 hardware), without the ESP32-C6. See CHANGES-v2fix.md for the full list, references and known limitations. Untested candidate: needs layout review before fabrication.
Parts:
- added C103: 100nF, Capacitor_SMD:C_0402_1005Metric, symbol Device:C
- added U16: SN74LV1T34DCKR, Package_TO_SOT_SMD:SOT-353_SC-70-5, symbol Logic_LevelTranslator:SN74LV1T34DCK
Connections:
- net +5V: now also C103.1, U16.5 (VCC)
- net ESP_WS2812: now also U16.2 (A); no longer LED1.3 (DIN)
- net GND: now also C103.2, U16.3 (GND)
- new net LED_DIN_5V: LED1.3 (DIN), U16.4 (Y)
- no-connect marks 1 -> 2
Changed lines of the file:
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@@
 	(wire
 		(pts
-			(xy 31.75 76.2) (xy 35.56 76.2)
+			(xy 182.88 81.28) (xy 182.88 83.82)
 		)
 		(stroke
@@
 	(wire
 		(pts
-			(xy 182.88 81.28) (xy 182.88 83.82)
+			(xy 143.51 80.01) (xy 143.51 81.28)
 		)
 		(stroke
@@
 	(wire
 		(pts
-			(xy 143.51 80.01) (xy 143.51 81.28)
+			(xy 100.33 76.2) (xy 110.49 76.2)
 		)
 		(stroke
@@
 	(wire
 		(pts
-			(xy 100.33 76.2) (xy 110.49 76.2)
+			(xy 34.29 88.9) (xy 34.29 91.44)
 		)
 		(stroke
@@
 	(wire
 		(pts
-			(xy 34.29 88.9) (xy 34.29 91.44)
+			(xy 143.51 71.12) (xy 143.51 72.39)
 		)
 		(stroke
@@
 	(wire
 		(pts
-			(xy 143.51 71.12) (xy 143.51 72.39)
+			(xy 219.71 71.12) (xy 222.25 71.12)
 		)
 		(stroke
@@
 	(wire
 		(pts
-			(xy 219.71 71.12) (xy 222.25 71.12)
+			(xy 100.33 81.28) (xy 102.87 81.28)
 		)
 		(stroke
@@
 	(wire
 		(pts
-			(xy 100.33 81.28) (xy 102.87 81.28)
+			(xy 140.97 81.28) (xy 143.51 81.28)
 		)
 		(stroke
@@
 	(wire
 		(pts
-			(xy 140.97 81.28) (xy 143.51 81.28)
+			(xy 222.25 71.12) (xy 222.25 68.58)
 		)
 		(stroke
@@
 	(wire
 		(pts
-			(xy 222.25 71.12) (xy 222.25 68.58)
+			(xy 222.25 81.28) (xy 222.25 83.82)
 		)
 		(stroke
@@
 	(wire
 		(pts
-			(xy 222.25 81.28) (xy 222.25 83.82)
+			(xy 222.25 71.12) (xy 222.25 72.39)
 		)
 		(stroke
@@
 	(wire
 		(pts
-			(xy 222.25 71.12) (xy 222.25 72.39)
+			(xy 140.97 71.12) (xy 143.51 71.12)
 		)
 		(stroke
@@
 	(wire
 		(pts
-			(xy 140.97 71.12) (xy 143.51 71.12)
+			(xy 102.87 71.12) (xy 102.87 72.39)
 		)
 		(stroke
@@
 	(wire
 		(pts
-			(xy 102.87 71.12) (xy 102.87 72.39)
+			(xy 182.88 71.12) (xy 182.88 68.58)
 		)
 		(stroke
@@
 	(wire
 		(pts
-			(xy 182.88 71.12) (xy 182.88 68.58)
+			(xy 233.68 78.74) (xy 234.95 78.74)
 		)
 		(stroke
@@
 	(wire
 		(pts
-			(xy 233.68 78.74) (xy 234.95 78.74)
+			(xy 143.51 81.28) (xy 143.51 83.82)
 		)
 		(stroke
@@
 	(wire
 		(pts
-			(xy 143.51 81.28) (xy 143.51 83.82)
+			(xy 255.27 78.74) (xy 257.81 78.74)
 		)
 		(stroke
@@
 	(wire
 		(pts
-			(xy 255.27 78.74) (xy 257.81 78.74)
+			(xy 34.29 78.74) (xy 35.56 78.74)
 		)
 		(stroke
@@
 	(wire
 		(pts
-			(xy 34.29 78.74) (xy 35.56 78.74)
+			(xy 180.34 71.12) (xy 182.88 71.12)
 		)
 		(stroke
@@
 	(wire
 		(pts
-			(xy 180.34 71.12) (xy 182.88 71.12)
+			(xy 58.42 78.74) (xy 58.42 81.28)
 		)
 		(stroke
@@
 	(wire
 		(pts
-			(xy 58.42 78.74) (xy 58.42 81.28)
+			(xy 257.81 78.74) (xy 257.81 81.28)
 		)
 		(stroke
@@
 	(wire
 		(pts
-			(xy 257.81 78.74) (xy 257.81 81.28)
+			(xy 102.87 80.01) (xy 102.87 81.28)
 		)
 		(stroke
 			(width 0)
 			(type default)
-		)
-	)
-	(wire
-		(pts
-			(xy 102.87 80.01) (xy 102.87 81.28)
-		)
-		(stroke
-			(width 0)
-			(type default)
-		)
-	)
-	(global_label "ESP_WS2812"
-		(shape input)
-		(at 31.75 76.2 180)
-		(fields_autoplaced yes)
-		(effects
-			(font
-				(size 1.27 1.27)
-			)
-			(justify right)
-		)
-		(property "Intersheetrefs" "${INTERSHEET_REFS}"
-			(at 16.6698 76.2 0)
-			(effects
-				(font
-					(size 1.27 1.27)
-				)
-				(justify right)
-				(hide yes)
-			)
 		)
 	)
@@
 		)
 	)
+	(wire (pts (xy 35.56 76.2) (xy 30.480000000000004 76.2)) (stroke (width 0) (type default)))
+	(label "LED_DIN_5V" (at 30.480000000000004 76.2 180) (fields_autoplaced yes) (effects (font (size 1.27 1.27)) (justify left bottom)))
+	(symbol
+		(lib_id "Logic_LevelTranslator:SN74LV1T34DCK")
+		(at 60.96 121.92 0)
+		(unit 1)
+		(exclude_from_sim no)
+		(in_bom yes)
+		(on_board yes)
+		(dnp no)
+		(property "Reference" "U16" (at 60.96 116.92 0) (effects (font (size 1.27 1.27))))
+		(property "Value" "SN74LV1T34DCKR" (at 60.96 126.92 0) (effects (font (size 1.27 1.27))))
+		(property "Footprint" "Package_TO_SOT_SMD:SOT-353_SC-70-5" (at 60.96 121.92 0) (effects (font (size 1.27 1.27)) (hide yes)))
+		(property "Datasheet" "~" (at 60.96 121.92 0) (effects (font (size 1.27 1.27)) (hide yes)))
+		(property "MPN" "SN74LV1T34DCKR" (at 60.96 121.92 0) (effects (font (size 1.27 1.27)) (hide yes)))
+		(property "Manufacturer" "Texas Instruments" (at 60.96 121.92 0) (effects (font (size 1.27 1.27)) (hide yes)))
+		(property "LCSC Part #" "C78541" (at 60.96 121.92 0) (effects (font (size 1.27 1.27)) (hide yes)))
+		(property "Description" "3.3V->5V level shift for SK6812 data" (at 60.96 121.92 0) (effects (font (size 1.27 1.27)) (hide yes)))
+		(property "Manufacturer Part" "SN74LV1T34DCKR" (at 60.96 121.92 0) (effects (font (size 1.27 1.27)) (hide yes)))
+		(pin "2")
+		(pin "1")
+		(pin "5")
+		(pin "3")
+		(pin "4")
+		(instances (project "nest-mini-v2-drop-in-pcb" (path "/204e071a-14ed-47a0-be54-332ac2b951cf/18f90dfa-9bd7-48d0-80c5-47366522e296" (reference "U16") (unit 1))))
+	)
+	(wire (pts (xy 53.34 121.92) (xy 48.260000000000005 121.92)) (stroke (width 0) (type default)))
+	(global_label "ESP_WS2812"
+		(shape input)
+		(at 48.260000000000005 121.92 180)
+		(fields_autoplaced yes)
+		(effects (font (size 1.27 1.27)) (justify right))
+		(property "Intersheetrefs" "${INTERSHEET_REFS}" (at 48.260000000000005 121.92 0) (effects (font (size 1.27 1.27)) (hide yes)))
+	)
+	(no_connect (at 55.88 119.38))
+	(wire (pts (xy 60.96 114.3) (xy 60.96 111.75999999999999)) (stroke (width 0) (type default)))
+	(symbol
+		(lib_id "power:+5V")
+		(at 60.96 111.75999999999999 0)
+		(unit 1)
+		(exclude_from_sim no)
+		(in_bom yes)
+		(on_board yes)
+		(dnp no)
+		(property "Reference" "#PWR0901" (at 60.96 106.75999999999999 0) (effects (font (size 1.27 1.27)) (hide yes)))
+		(property "Value" "+5V" (at 60.96 116.75999999999999 0) (effects (font (size 1.27 1.27))))
+		(property "Footprint" "" (at 60.96 111.75999999999999 0) (effects (font (size 1.27 1.27)) (hide yes)))
+		(property "Datasheet" "~" (at 60.96 111.75999999999999 0) (effects (font (size 1.27 1.27)) (hide yes)))
+		(pin "1")
+		(instances (project "nest-mini-v2-drop-in-pcb" (path "/204e071a-14ed-47a0-be54-332ac2b951cf/18f90dfa-9bd7-48d0-80c5-47366522e296" (reference "#PWR0901") (unit 1))))
+	)
+	(wire (pts (xy 60.96 129.54) (xy 60.96 132.07999999999998)) (stroke (width 0) (type default)))
+	(symbol
+		(lib_id "power:GND")
+		(at 60.96 132.07999999999998 0)
+		(unit 1)
+		(exclude_from_sim no)
+		(in_bom yes)
+		(on_board yes)
+		(dnp no)
+		(property "Reference" "#PWR0902" (at 60.96 127.07999999999998 0) (effects (font (size 1.27 1.27)) (hide yes)))
+		(property "Value" "GND" (at 60.96 137.07999999999998 0) (effects (font (size 1.27 1.27))))
+		(property "Footprint" "" (at 60.96 132.07999999999998 0) (effects (font (size 1.27 1.27)) (hide yes)))
+		(property "Datasheet" "~" (at 60.96 132.07999999999998 0) (effects (font (size 1.27 1.27)) (hide yes)))
+		(pin "1")
+		(instances (project "nest-mini-v2-drop-in-pcb" (path "/204e071a-14ed-47a0-be54-332ac2b951cf/18f90dfa-9bd7-48d0-80c5-47366522e296" (reference "#PWR0902") (unit 1))))
+	)
+	(wire (pts (xy 68.58 121.92) (xy 73.66 121.92)) (stroke (width 0) (type default)))
+	(label "LED_DIN_5V" (at 73.66 121.92 0) (fields_autoplaced yes) (effects (font (size 1.27 1.27)) (justify left bottom)))
+	(symbol
+		(lib_id "Device:C")
+		(at 81.28 121.92 0)
+		(unit 1)
+		(exclude_from_sim no)
+		(in_bom yes)
+		(on_board yes)
+		(dnp no)
+		(property "Reference" "C103" (at 81.28 116.92 0) (effects (font (size 1.27 1.27))))
+		(property "Value" "100nF" (at 81.28 126.92 0) (effects (font (size 1.27 1.27))))
+		(property "Footprint" "Capacitor_SMD:C_0402_1005Metric" (at 81.28 121.92 0) (effects (font (size 1.27 1.27)) (hide yes)))
+		(property "Datasheet" "~" (at 81.28 121.92 0) (effects (font (size 1.27 1.27)) (hide yes)))
+		(property "Manufacturer Part" "CL05B104KO5NNNC" (at 81.28 121.92 0) (effects (font (size 1.27 1.27)) (hide yes)))
+		(property "LCSC Part #" "C1525" (at 81.28 121.92 0) (effects (font (size 1.27 1.27)) (hide yes)))
+		(pin "1")
+		(pin "2")
+		(instances (project "nest-mini-v2-drop-in-pcb" (path "/204e071a-14ed-47a0-be54-332ac2b951cf/18f90dfa-9bd7-48d0-80c5-47366522e296" (reference "C103") (unit 1))))
+	)
+	(wire (pts (xy 81.28 118.11) (xy 81.28 115.57)) (stroke (width 0) (type default)))
+	(symbol
+		(lib_id "power:+5V")
+		(at 81.28 115.57 0)
+		(unit 1)
+		(exclude_from_sim no)
+		(in_bom yes)
+		(on_board yes)
+		(dnp no)
+		(property "Reference" "#PWR0903" (at 81.28 110.57 0) (effects (font (size 1.27 1.27)) (hide yes)))
+		(property "Value" "+5V" (at 81.28 120.57 0) (effects (font (size 1.27 1.27))))
+		(property "Footprint" "" (at 81.28 115.57 0) (effects (font (size 1.27 1.27)) (hide yes)))
+		(property "Datasheet" "~" (at 81.28 115.57 0) (effects (font (size 1.27 1.27)) (hide yes)))
+		(pin "1")
+		(instances (project "nest-mini-v2-drop-in-pcb" (path "/204e071a-14ed-47a0-be54-332ac2b951cf/18f90dfa-9bd7-48d0-80c5-47366522e296" (reference "#PWR0903") (unit 1))))
+	)
+	(wire (pts (xy 81.28 125.73) (xy 81.28 128.27)) (stroke (width 0) (type default)))
+	(symbol
+		(lib_id "power:GND")
+		(at 81.28 128.27 0)
+		(unit 1)
+		(exclude_from_sim no)
+		(in_bom yes)
+		(on_board yes)
+		(dnp no)
+		(property "Reference" "#PWR0904" (at 81.28 123.27000000000001 0) (effects (font (size 1.27 1.27)) (hide yes)))
+		(property "Value" "GND" (at 81.28 133.27 0) (effects (font (size 1.27 1.27))))
+		(property "Footprint" "" (at 81.28 128.27 0) (effects (font (size 1.27 1.27)) (hide yes)))
+		(property "Datasheet" "~" (at 81.28 128.27 0) (effects (font (size 1.27 1.27)) (hide yes)))
+		(pin "1")
+		(instances (project "nest-mini-v2-drop-in-pcb" (path "/204e071a-14ed-47a0-be54-332ac2b951cf/18f90dfa-9bd7-48d0-80c5-47366522e296" (reference "#PWR0904") (unit 1))))
+	)
 )
