File: nest-mini-v2-drop-in-pcb.kicad_pcb (KiCad board)
At the start: 4 copper layers, 74.5 x 70.6 mm, 238 parts, among them J1 usb_c, J2 Conn_01x05, J3 XTAG DEV, J4 XMOS JTAG, J5 1775443-2, Q1 LBSS138WT1G, Q2 LBSS138WT1G, Q3 BC847B, SW1 Reset, SW2 BOOT, U1 CUS-12TB, U10 XU316-1024-QF60B-C24​, U11 W25Q32JVSSIQ, U12 SN74LVC125APWR, U13 TLV73333PDBVR, U14 TAS5805MPWPR, U15 MPR121QR2, U2 TS3USB221ERSER, U3 TPS62130, U4 AP22802AW5-7, U5 MIC5365-1.8YC5-TR, U6 TPS7A0309PDBVR, U7 TPS62130, U8 ESP32-S3R8, U9 W25Q128JVSIQ, X1 24MHz 12pF, Y1 40MHz

Commit message: v2-fix: issue #53 fixes on the v2 hardware (XMOS 0.9V buck, Voice PE I2S roles, U12, JTAG header, TAS5805M ADR, LED level shift, routing bugs)
Based on 7de6eec (v2 hardware), without the ESP32-C6. See CHANGES-v2fix.md for the full list, references and known limitations. Untested candidate: needs layout review before fabrication.
Parts:
- removed J3: XTAG DEV, Connector_PinHeader_2.54mm:PinHeader_1x04_P2.54mm_Vertical
- added C100: 22pF, Capacitor_SMD:C_0402_1005Metric, F.Cu at (148.4, 84.2)
- added C101: 10uF, Capacitor_SMD:C_0603_1608Metric, F.Cu at (148.6, 78.5)
- added C102: 10uF, Capacitor_SMD:C_0603_1608Metric, F.Cu at (145.7, 84.9)
- added C103: 100nF, Capacitor_SMD:C_0402_1005Metric, F.Cu at (103.9, 94.7)
- added L8: 1uH, Inductor_SMD:L_Murata_DFE201610P, F.Cu at (145.7, 81.7)
- added R74: 51k, Resistor_SMD:R_0402_1005Metric, F.Cu at (148.4, 83.2)
- added R75: 100k, Resistor_SMD:R_0402_1005Metric, F.Cu at (148.4, 85.2)
- added U16: SN74LV1T34DCKR, Package_TO_SOT_SMD:SOT-353_SC-70-5, F.Cu at (103.3, 92.7)
- C18: value 4.7uF -> 10uF
- C44: value 1uF -> 10uF
- FB3: value 600R -> 120R
- J4: value XMOS JTAG -> XTAG JTAG (xSYS2 pins 1-10); footprint Connector_PinHeader_2.54mm:PinHeader_2x05_P2.54mm_Vertical -> Connector_PinHeader_1.27mm:PinHeader_2x05_P1.27mm_Vertical
- R70: value 0R -> 15k
- U6: value TPS7A0309PDBVR -> TPS62065DSGR; footprint Package_TO_SOT_SMD:SOT-23-5 -> Package_SON:Texas_DSG0008A_WSON-8-1EP_2x2mm_P0.5mm_EP0.9x1.6mm
- moved J4 23.2 mm to (151.9, 94.4), turned to 90 degrees
- moved U6 12.7 mm to (148.6, 80.7), turned to 0 degrees
Connections:
- J4 pad 1: /XMOS/RST_N -> +1V8
- J4 pad 10: (no net) -> /XMOS/RST_N
- J4 pad 2: GND -> /XMOS/TMS
- J4 pad 3: /XMOS/TDI -> GND
- J4 pad 4: +5V -> /XMOS/TCK
- J4 pad 5: /XMOS/TDO -> GND
- J4 pad 6: VDDIO -> /XMOS/TDO
- J4 pad 7: /XMOS/TCK -> GND
- J4 pad 8: GND -> /XMOS/TDI
- J4 pad 9: /XMOS/TMS -> GND
- LED1 pad 3: ESP_WS2812 -> /LEDs/LED_DIN_5V
- R37 pad 2: /XMOS/XL_UP0 -> unconnected-(R37-Pad2)
- R38 pad 2: /XMOS/XL_UP1 -> unconnected-(R38-Pad2)
- R70 pad 1: GNDA -> DVDD
- U10 pad 10: unconnected-(U10-X1D01-Pad10) -> I2S_LRCK
- U10 pad 13: unconnected-(U10-X1D10-Pad13) -> I2S_BCLK
- U10 pad 14: /XMOS/MIC_DATA_2 -> I2S_MCLK
- U10 pad 33: /XMOS/XL_DN1 -> unconnected-(U10-X1D16-Pad33)
- U10 pad 35: /XMOS/XL_DN0 -> unconnected-(U10-X1D17-Pad35)
- U10 pad 53: unconnected-(U10-X1D34-Pad53) -> I2S_DIN_ESP
- U12 pad 1: /XMOS/MIC_DATA_M_2 -> GND
- U12 pad 2: MUTE_ON -> GND
- U12 pad 3: /XMOS/MIC_DATA_2 -> unconnected-(U12-1Y-Pad3)
- U6 pad 1: +3V3 -> GND
- U6 pad 2: GND -> /Power/SW_0V9
- U6 pad 3: +3V3 -> GND
- U6 pad 4: (no net) -> /Power/FB_0V9
- U6 pad 5: +0V9 -> +5V
Routing:
- net +0V9: track 17.6 -> 54.0 mm, vias 0 -> 2
- net Net-(U15-ELEC1): track 0.00 -> 35.2 mm, vias 0 -> 2
- net +1V8: track 40.0 -> 71.4 mm, vias 5 -> 7
- net I2S_LRCK: track 31.9 -> 61.8 mm, vias 0 -> 5
- net /ESP32-S3R8/TOUCH_IRQ: track 0.00 -> 28.2 mm, vias 0 -> 3
- net /XMOS/RST_N: track 54.5 -> 82.2 mm, vias 2 -> 4
- net /XMOS/XL_UP1: track 27.6 -> 0.00 mm, vias 2 -> 0
- net /XMOS/XL_DN0: track 26.5 -> 0.00 mm, vias 2 -> 0
- net /XMOS/XL_DN1: track 25.4 -> 0.00 mm, vias 2 -> 0
- net /XMOS/XL_UP0: track 24.8 -> 0.00 mm, vias 2 -> 0
- net /ESP32-S3R8/SPI_HD: track 25.4 -> 6.91 mm, vias 0 -> 2
- net I2S_MCLK: track 1.05 -> 17.7 mm, vias 0 -> 5
- net I2S_BCLK: track 32.4 -> 48.2 mm, vias 2 -> 5
- net /XMOS/MIC_DATA_2: track 12.5 -> 0.00 mm, vias 2 -> 0
- net /XMOS/TCK: track 49.6 -> 39.6 mm, vias 0 -> 1
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Other:
- board text removed: "1"
- board text removed: "10"
- board text removed: "4"
- board text removed: "9"
