File: nest-mini-v2-drop-in-pcb.kicad_pcb (KiCad board)
At the start: 4 copper layers, 74.5 x 70.6 mm, 245 parts, among them J1 usb_c, J2 Conn_01x05, J4 XTAG JTAG (xSYS2 pins 1-10), J5 1775443-2, Q1 LBSS138WT1G, Q2 LBSS138WT1G, Q3 BC847B, SW1 Reset, SW2 BOOT, U1 CUS-12TB, U10 XU316-1024-QF60B-C24​, U11 W25Q32JVSSIQ, U12 SN74LVC125APWR, U13 TLV73333PDBVR, U14 TAS5805MPWPR, U15 MPR121QR2, U16 SN74LV1T34DCKR, U2 TS3USB221ERSER, U3 TPS62130, U4 AP22802AW5-7, U5 MIC5365-1.8YC5-TR, U6 TPS62065DSGR, U7 TPS62130, U8 ESP32-S3R8, U9 W25Q128JVSIQ, X1 24MHz 12pF, Y1 40MHz

Commit message: v2.1: octilinear re-route of added tracks, bundled JTAG, TI-style buck layout, v2.1 silkscreen
All tracks added in v2-fix re-routed at 0/45/90 deg with no mid-trace splits; branches only at pads or vias. JTAG runs as one parallel bundle (J4 moved to the top side). Buck converter re-laid with power polygons. XU316_RST moved to GPIO21, LED data to GPIO4, X1D11 MCLK left unconnected; MiciMike.yaml updated to match. Silkscreen and title blocks now say v2.1. KiCad 9 DRC with schematic parity shows only the items already on the v2 board. See CHANGES-v2fix.md.

Co-Authored-By: Claude Opus 5.5 <noreply@anthropic.com>
Claude-Session: https://claude.ai/code/session_01DBYfebaHp5UuC2Xws8yAJw
Parts:
- J4: moved to F.Cu
- moved J4 5.08 mm to (146.9, 94.4)
- moved L8 0.53 mm to (145.7, 81.2)
- moved C101 0.17 mm to (148.4, 78.5)
- moved C102 0.07 mm to (145.7, 85.0)
- moved C100 0.06 mm to (148.5, 84.2)
- turned U16 to 180 degrees
Connections:
- U10 pad 14: I2S_MCLK -> unconnected-(U10-X1D11-Pad14)
- U8 pad 23: XU316_RST -> unconnected-(U8-GPIO17-Pad23)
- U8 pad 27: ESP_WS2812 -> XU316_RST
- U8 pad 9: unconnected-(U8-GPIO4-Pad9) -> ESP_WS2812
Routing:
- net +1V8: track 71.4 -> 98.8 mm, vias 7 -> 5
- net /XMOS/TCK: track 39.6 -> 58.4 mm, vias 1 -> 2
- net I2S_LRCK: track 61.8 -> 78.9 mm, vias 5 -> 3
- net I2S_MCLK: track 17.7 -> 1.05 mm, vias 5 -> 0
- net Net-(U15-ELEC1): track 35.2 -> 51.7 mm, vias 2 -> 4
- net /XMOS/TDI: track 44.0 -> 60.4 mm, vias 8 -> 1
- net /XMOS/TMS: track 49.5 -> 61.0 mm
- net /ESP32-S3R8/TOUCH_IRQ: track 28.2 -> 38.1 mm
- net /XMOS/TDO: track 52.1 -> 60.1 mm, vias 4 -> 1
- net ESP_WS2812: track 41.7 -> 35.0 mm
- net I2S_BCLK: track 48.2 -> 52.7 mm
- net /XMOS/RST_N: track 82.2 -> 78.5 mm, vias 4 -> 1
- net GND: track 6.75 -> 3.65 mm, vias 179 -> 177
- net /LEDs/LED_DIN_5V: track 5.74 -> 2.85 mm
- net +5V: track 72.0 -> 69.8 mm, vias 18 -> 16
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- added copper zone on F.Cu, net +0V9
- added copper zone on F.Cu, net +5V
- added copper zone on F.Cu, net /Power/SW_0V9
Other:
- board text added: "MiciMike Nest mini (Gen2) drop-in PCB v2.1"
- board text removed: "MiciMike Nest mini (Gen2) drop-in PCB"
