File: power_handling.kicad_sch (KiCad schematic)
At the start: 64 parts, among them J1 usb_c, U1 CUS-12TB, U2 TS3USB221ERSER, U3 TPS62130, U4 AP22802AW5-7, U5 MIC5365-1.8YC5-TR, U6 TPS7A0309PDBVR, U7 TPS62130

Commit message: v2-fix: issue #53 fixes on the v2 hardware (XMOS 0.9V buck, Voice PE I2S roles, U12, JTAG header, TAS5805M ADR, LED level shift, routing bugs)
Based on 7de6eec (v2 hardware), without the ESP32-C6. See CHANGES-v2fix.md for the full list, references and known limitations. Untested candidate: needs layout review before fabrication.
Parts:
- removed U6: TPS7A0309PDBVR, Package_TO_SOT_SMD:SOT-23-5, symbol New_Library:MIC5365-1.8YC5-TR
- added C100: 22pF, Capacitor_SMD:C_0402_1005Metric, symbol Device:C
- added C101, C102: 10uF, Capacitor_SMD:C_0603_1608Metric, symbol Device:C
- added L8: 1uH, Inductor_SMD:L_Murata_DFE201610P, symbol Device:L
- added R74: 51k, Resistor_SMD:R_0402_1005Metric, symbol Device:R
- added R75: 100k, Resistor_SMD:R_0402_1005Metric, symbol Device:R
- added U6: TPS62065DSGR, Package_SON:Texas_DSG0008A_WSON-8-1EP_2x2mm_P0.5mm_EP0.9x1.6mm, symbol MiciMike:TPS62065DSGR
- C18: value 4.7uF -> 10uF; LCSC Part # C913474 -> C19702; Manufacturer Part GRM188Z71A475KE15D -> CL10A106KP8NNNC; Supplier Part C913474 -> C19702
- U2: LCSC Part # (none) -> C129313; Manufacturer Part (none) -> TS3USB221ERSER
Connections:
- net +0V9: now also C100.1, C102.1, L8.2, R74.1
- net +5V: now also C101.1, U6.5 (EN), U6.6 (MODE), U6.7 (AVIN), U6.8 (PVIN)
- net GND: now also C101.2, C102.2, R75.2, U6.1 (PGND), U6.3 (AGND), U6.9 (PAD)
- new net FB_0V9: C100.2, R74.2, R75.1, U6.4 (FB)
- new net SW_0V9: L8.1, U6.2 (SW)
