File: xmos.kicad_sch (KiCad schematic)
At the start: 84 parts, among them J3 XTAG DEV, J4 XMOS JTAG, Q1 LBSS138WT1G, Q2 LBSS138WT1G, Q3 BC847B, U10 XU316-1024-QF60B-C24​, U11 W25Q32JVSSIQ, U12 SN74LVC125APWR, U13 TLV73333PDBVR, X1 24MHz 12pF

Commit message: v2-fix: issue #53 fixes on the v2 hardware (XMOS 0.9V buck, Voice PE I2S roles, U12, JTAG header, TAS5805M ADR, LED level shift, routing bugs)
Based on 7de6eec (v2 hardware), without the ESP32-C6. See CHANGES-v2fix.md for the full list, references and known limitations. Untested candidate: needs layout review before fabrication.
Parts:
- removed J3: XTAG DEV, Connector_PinHeader_2.54mm:PinHeader_1x04_P2.54mm_Vertical, symbol Connector:Conn_01x04_Pin
- removed J4: XMOS JTAG, Connector_PinHeader_2.54mm:PinHeader_2x05_P2.54mm_Vertical, symbol Connector_Generic_MountingPin:Conn_2Rows-09Pins_MountingPin
- added J4: XTAG JTAG (xSYS2 pins 1-10), Connector_PinHeader_1.27mm:PinHeader_2x05_P1.27mm_Vertical, symbol Connector_Generic:Conn_02x05_Odd_Even
- C44: value 1uF -> 10uF; LCSC Part # C52923 -> C15525; Manufacturer Part CL05A105KA5NQNC -> CL05A106MQ5NUNC; Supplier Part C52923 -> C15525; Voltage 25V -> 6.3V
- FB3: value 600R -> 120R; Current 500mA -> 2A; LCSC Part # C85833 -> C14709; MP BLM18KG601SN1D -> BLM18PG121SN1D; MPN (none) -> BLM18PG121SN1D; Manufacturer Part BLM18KG601SN1D -> BLM18PG121SN1D; Part number BLM18KG601SN1D -> BLM18PG121SN1D; Supplier Part C85833 -> C14709
- MK3, R37, R38, R61, R64: now not fitted
- U11: LCSC Part # (none) -> C179173; Manufacturer Part (none) -> W25Q32JVSSIQ
Connections:
- net +1V8: now also J4.1 (Pin_1)
- net GND: now also U12.1 (1~{OE}), U12.2 (1A), J4.3 (Pin_3), J4.5 (Pin_5), J4.7 (Pin_7), J4.9 (Pin_9)
- net MIC_DATA_M_2: no longer U12.1 (1~{OE})
- net MUTE_ON: no longer U12.2 (1A)
- net RST_N: now also J4.10 (Pin_10)
- net TCK: now also J4.4 (Pin_4)
- net TDI: now also J4.8 (Pin_8)
- net TDO: now also J4.6 (Pin_6)
- net TMS: now also J4.2 (Pin_2)
- net I2S_LRCK: now reaches U10.10 (X1D01)
- net I2S_BCLK: now reaches U10.13 (X1D10)
- net I2S_DIN_ESP: now reaches U10.53 (X1D34)
- net MIC_DATA_2: no longer names the net of U12.3 (1Y)
- net MIC_DATA_2: no longer U10.14 (X1D11)
- net XL_DN0: no longer names the net of U10.35 (X1D17)
- net XL_DN1: no longer names the net of U10.33 (X1D16)
- net XL_UP0: no longer names the net of R37.2
- net XL_UP1: no longer names the net of R38.2
- new net I2S_MCLK: U10.14 (X1D11)
- no-connect marks 10 -> 12
